File: Glider_Revision.kicad_sch (KiCad schematic)
At the start: 20 parts, among them J1 ESP32 Right, J10 Light Enable, J2 ESP32 Left, J3 MPU-6050, J4 GT-U7, J5 GY-271 QMC5883L, J6 LiPo 7.4, J7 ServoLeft, J8 ServoRight, J9 Light Power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

Commit message: Schemnatic updates
Parts:
- added H1, H2, H3, H4: MountingHole, MountingHole:MountingHole_2.5mm_Pad, symbol Mechanical:MountingHole
- added S1: MS0850502F030P1A, custom:SW_MS0850502F030P1A, symbol custom:MS0850502F030P1A
- C5: footprint (none) -> Capacitor_THT:CP_Radial_D4.0mm_P2.00mm
- J1, J2: footprint Connector_PinHeader_1.00mm:PinHeader_1x20_P1.00mm_Vertical -> Connector_PinHeader_2.54mm:PinHeader_1x19_P2.54mm_Vertical
- J10, J9: footprint Connector_PinHeader_1.00mm:PinHeader_1x02_P1.00mm_Vertical -> Connector_PinHeader_2.54mm:PinHeader_1x02_P2.54mm_Horizontal
- J3: footprint Connector_PinHeader_1.00mm:PinHeader_1x08_P1.00mm_Vertical -> Connector_PinHeader_2.54mm:PinHeader_1x08_P2.54mm_Vertical
- J4, J5: footprint Connector_PinHeader_1.00mm:PinHeader_1x05_P1.00mm_Vertical -> Connector_PinHeader_2.54mm:PinHeader_1x05_P2.54mm_Vertical
- J6: footprint Connector_PinHeader_1.00mm:PinHeader_1x02_P1.00mm_Vertical -> Connector_PinSocket_2.54mm:PinSocket_1x02_P2.54mm_Vertical
- J7, J8: footprint (none) -> Connector_PinHeader_2.54mm:PinHeader_1x03_P2.54mm_Vertical
- U1: footprint Package_TO_SOT_THT:TO-3P-3_Vertical -> Package_TO_SOT_THT:TO-220-3_Vertical
Connections:
- net GND: now also S1.1
- net GPIO11: now also S1.3
- net GPIO34: now also S1.2
- no-connect marks 1 -> 39

Commit message: Updates
Parts:
- removed S1: MS0850502F030P1A, custom:SW_MS0850502F030P1A, symbol custom:MS0850502F030P1A
- added J11: Limit Switch connector, Connector_PinHeader_2.54mm:PinHeader_1x03_P2.54mm_Vertical, symbol Connector:Conn_01x03_Pin
- J10, J9: footprint Connector_PinHeader_2.54mm:PinHeader_1x02_P2.54mm_Horizontal -> Connector_PinHeader_2.54mm:PinHeader_1x02_P2.54mm_Vertical
- J5: value GY-271 QMC5883L -> MMC5603
Connections:
- net DRDY_mag is gone; now on net GPIO21_I2C_SDA: J5.1 (Pin_1)
- net GND: now also J5.3 (Pin_3), J11.1 (Pin_1); no longer J5.4 (Pin_4)
- net GPIO11: now also J11.3 (Pin_3)
- net GPIO21_I2C_SDA: no longer J5.2 (Pin_2)
- net GPIO22_I2C_SCL: now also J5.2 (Pin_2); no longer J5.3 (Pin_3)
- net GPIO34: now also J11.2 (Pin_2)
- no-connect marks 39 -> 38
