File: Glider_Revision.kicad_pcb (KiCad board)
At the start: 2 copper layers, 55.5 x 89.6 mm, 25 parts, among them J1 ESP32 Right, J10 Light Enable, J2 ESP32 Left, J3 MPU-6050, J4 GT-U7, J5 GY-271 QMC5883L, J6 LiPo 7.4, J7 ServoLeft, J8 ServoRight, J9 Light Power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

Commit message: Updates
Parts:
- removed S1: MS0850502F030P1A, custom:SW_MS0850502F030P1A
- added J11: Limit Switch connector, Connector_PinHeader_2.54mm:PinHeader_1x03_P2.54mm_Vertical, F.Cu at (108.2, 107.5)
- J10, J9: footprint Connector_PinHeader_2.54mm:PinHeader_1x02_P2.54mm_Horizontal -> Connector_PinHeader_2.54mm:PinHeader_1x02_P2.54mm_Vertical
- J5: value GY-271 QMC5883L -> MMC5603
- moved H1 29.1 mm to (123.2, 63.3)
- moved H2 22.6 mm to (123.5, 47.8)
- moved J9 3.85 mm to (111.7, 47.4), turned to 0 degrees
- moved J10 0.70 mm to (134.8, 50.1), turned to 180 degrees
Connections:
- J5 pad 1: /DRDY_mag -> /GPIO21_I2C_SDA
- J5 pad 2: /GPIO21_I2C_SDA -> /GPIO22_I2C_SCL
- J5 pad 3: /GPIO22_I2C_SCL -> GND
- J5 pad 4: GND -> unconnected-(J5-Pin_4-Pad4)
Other:
- board size 55.5 x 89.6 mm -> 55.5 x 73.5 mm
- board text added: "GT-U7"
- board text added: "L7805CV"
- board text added: "MMC5603"
- board text added: "MPU-6050"
- board text added: "NC,34"
- board text added: "NO,11"
- board text added: "PROG, 15"
- board text added: "RX"
- board text added: "SCL"
- board text added: "SDA"
- board text added: "SrvL"
- board text added: "SrvR"
- board text added: "TX"
- board text removed: "ESP_PWM(GPIO15)"

Commit message: Schemnatic updates
Routing:
- net GND: track 0.00 -> 240.7 mm, vias 0 -> 30
- net /3_3V: track 0.00 -> 133.1 mm, vias 0 -> 8
- net /Vin: track 0.00 -> 125.9 mm, vias 0 -> 2
- net /5V: track 0.00 -> 118.4 mm, vias 0 -> 10
- net /GPIO11: track 0.00 -> 85.8 mm, vias 0 -> 4
- net /GPIO21_I2C_SDA: track 0.00 -> 67.0 mm, vias 0 -> 4
- net /GPIO22_I2C_SCL: track 0.00 -> 47.6 mm, vias 0 -> 4
- net /GPIO34: track 0.00 -> 45.5 mm, vias 0 -> 2
- net /GPIO25: track 0.00 -> 37.7 mm, vias 0 -> 2
- net /GPIO15: track 0.00 -> 35.9 mm, vias 0 -> 4
- net /GPIO26: track 0.00 -> 30.6 mm, vias 0 -> 3
- net /GPIO17_TX2: track 0.00 -> 22.7 mm, vias 0 -> 2
- net /GPIO16_RX2: track 0.00 -> 22.4 mm, vias 0 -> 2
